Commit message: create a melodic branch

File: description/urdf/robot.urdf (robot description, URDF)
Before this commit: robot robot, 3 links, 2 joints
Joints:
- joint fixed: origin (none) -> xyz=0 0 0 rpy=0 0 0
- joint joint1: origin xyz=0.0 0.0 4.0 rpy=0.0 0.0 0.0 -> xyz=0.0 0.0 2.00 rpy=0.0 0.0 0.0
